File: Kicad/Linear_Acuator_Control/Linear_Acuator_Control.kicad_sch (KiCad schematic)
At the start: 10 parts, among them K1 RT42xAxx, K3 RT42xAxx, Q1 IRLB3813, Q2 IRLB3813, U1 ESP32-S3-WROOM

Commit message: changing things to fix problems
Parts:
- added D3, D4: 1N4148WT, Diode_SMD:D_SOD-523, symbol Diode:1N4148WT
- added Q3, Q4: NMOS_Substrate, symbol Simulation_SPICE:NMOS_Substrate
- added R1, R3: 1k, Resistor_THT:R_Axial_DIN0207_L6.3mm_D2.5mm_P10.16mm_Horizontal, symbol PCM_SL_Resistors:1k
- added R2, R4: 10k, Resistor_THT:R_Axial_DIN0207_L6.3mm_D2.5mm_P10.16mm_Horizontal, symbol PCM_SL_Resistors:10k
- added R5, R6: 220, Resistor_THT:R_Axial_DIN0207_L6.3mm_D2.5mm_P10.16mm_Horizontal, symbol PCM_SL_Resistors:1k
Connections:
- net +24V: now also K1.A1, K3.A1, D3.1 (K)
- net Dir L1: now also R1.1; no longer K3.A1
- net Dir L2: now also R3.1; no longer K1.A1
- net GND: now also Q3.3 (S), Q3.4 (Bulk), Q4.3 (S), Q4.4 (Bulk), R2.2, R4.2; no longer K1.A2, K3.A2
- net Speed L1: now also R6.1; no longer Q1.1 (G)
- net Speed L2: now also R5.1; no longer Q2.1 (G)
- new net: Q1.1 (G), R6.2
- new net: D3.2 (A), K3.A2, Q3.1 (D)
- new net: Q3.2 (G), R1.2, R2.1
- new net: Q4.2 (G), R3.2, R4.1
- new net: D4.2 (A), K1.A2, Q4.1 (D)
- new net: Q2.1 (G), R5.2
Other:
- moved on the sheet: L3
