File: Kicad/Linear_Acuator_Control/Linear_Acuator_Control.kicad_sch (KiCad schematic)
At the start: 20 parts, among them K1 RT42xAxx, K3 RT42xAxx, Q1 IRLB3813, Q2 IRLB3813, Q3 2N7002, Q5 2N7002, U1 ESP32-S3-WROOM

Commit message: push to github, missing easyeda files atm
Parts:
- D1, D2: footprint Package_TO_SOT_THT:TO-220-2_Vertical -> Diode_SMD:D_SMB
- D3, D4: footprint Diode_SMD:D_SOD-523 -> Diode_SMD:D_SOD-123
- K1, K3, L1, L2, U1: now not fitted
- Q1, Q2: footprint Package_TO_SOT_THT:TO-220-3_Vertical -> Package_TO_SOT_SMD:SOT-23
- R6: footprint Resistor_THT:R_Axial_DIN0207_L6.3mm_D2.5mm_P10.16mm_Horizontal -> Resistor_SMD:R_0603_1608Metric
Connections:
- net L1SwitchedLow is gone; now on net GND: D1.2 (A), K3.11, Q1.2 (D)
- net Dir L1: now also Q3.1 (G), R1.2, R2.1
- net GND: now also D2.2 (A), K1.11, Q2.2 (D), Q5.1 (G), R3.2, R4.1
- net Net-(Q3-G): no longer Q3.1 (G), R1.2, R2.1
- net Net-(Q5-G): no longer Q5.1 (G), R3.2, R4.1
- net Speed L1: now also Q1.1 (G), R6.2; no longer R6.1
- new net Net-(Q1-G): R6.1
Changed lines of the file:
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@@
 		)
 	)
-	(label "Net-(Q5-G)"
+	(label "GND"
 		(at 143.51 57.15 180)
+		(effects
+			(font
+				(size 1.27 1.27)
+			)
+			(justify right bottom)
+		)
+	)
+	(label "Speed L1"
+		(at 160.02 60.96 0)
+		(effects
+			(font
+				(size 1.27 1.27)
+			)
+			(justify left bottom)
+		)
+	)
+	(label "GND"
+		(at 187.96 85.09 180)
 		(effects
 			(font
@@
 		)
 	)
-	(label "L1SwitchedLow"
-		(at 187.96 85.09 180)
-		(effects
-			(font
-				(size 1.27 1.27)
-			)
-			(justify right bottom)
-		)
-	)
 	(label "Dir L1"
 		(at 55.88 71.12 180)
@@
 		)
 	)
-	(label "Net-(Q3-G)"
+	(label "GND"
+		(at 240.03 92.71 180)
+		(effects
+			(font
+				(size 1.27 1.27)
+			)
+			(justify right bottom)
+		)
+	)
+	(label "Dir L1"
 		(at 143.51 88.9 180)
 		(effects
@@
 		)
 	)
-	(global_label "Speed L1"
+	(global_label "Net-(Q1-G)"
 		(shape input)
 		(at 138.43 60.96 180)
@@
 			)
 		)
-		(property "Footprint" "Resistor_THT:R_Axial_DIN0207_L6.3mm_D2.5mm_P10.16mm_Horizontal"
+		(property "Footprint" "Resistor_SMD:R_0603_1608Metric"
 			(at 157.099 65.278 0)
 			(hide yes)
@@
 			)
 		)
-		(property "Footprint" "Diode_SMD:D_SOD-523"
+		(property "Footprint" "Diode_SMD:D_SOD-123"
 			(at 163.195 71.12 0)
 			(hide yes)
@@
 		(on_board yes)
 		(in_pos_files yes)
-		(dnp no)
+		(dnp yes)
 		(property "Reference" "L1"
 			(at 190.5 46.9899 90)
@@
 			)
 		)
-		(property "Footprint" "Package_TO_SOT_THT:TO-220-3_Vertical"
+		(property "Footprint" "Package_TO_SOT_SMD:SOT-23"
 			(at 190.5 92.075 0)
 			(hide yes)
@@
 		(on_board yes)
 		(in_pos_files yes)
-		(dnp no)
+		(dnp yes)
 		(fields_autoplaced yes)
 		(property "Reference" "K3"
@@
 			)
 		)
-		(property "Footprint" "Package_TO_SOT_THT:TO-220-2_Vertical"
+		(property "Footprint" "Diode_SMD:D_SMB"
 			(at 243.84 88.265 0)
 			(hide yes)
@@
 		(on_board yes)
 		(in_pos_files yes)
-		(dnp no)
+		(dnp yes)
 		(fields_autoplaced yes)
 		(property "Reference" "U1"
@@
 		(on_board yes)
 		(in_pos_files yes)
-		(dnp no)
+		(dnp yes)
 		(fields_autoplaced yes)
 		(property "Reference" "K1"
@@
 			)
 		)
-		(property "Footprint" "Diode_SMD:D_SOD-523"
+		(property "Footprint" "Diode_SMD:D_SOD-123"
 			(at 213.995 69.85 0)
 			(hide yes)
@@
 			)
 		)
-		(property "Footprint" "Package_TO_SOT_THT:TO-220-2_Vertical"
+		(property "Footprint" "Diode_SMD:D_SMB"
 			(at 191.77 80.645 0)
 			(hide yes)
@@
 			)
 		)
-		(property "Footprint" "Package_TO_SOT_THT:TO-220-3_Vertical"
+		(property "Footprint" "Package_TO_SOT_SMD:SOT-23"
 			(at 240.03 99.695 0)
 			(hide yes)
@@
 		(on_board yes)
 		(in_pos_files yes)
-		(dnp no)
+		(dnp yes)
 		(property "Reference" "L2"
 			(at 240.03 46.9899 90)
